File: hav_node/hav_adxl345.kicad_sch (KiCad schematic)
At the start: 12 parts, among them U2 ADXL345BCCZ-RL7

Commit message: Rapihin skematik HAV
Other:
- note added: "TEST POINT SENSOR"
- note removed: "K-16.2 | TEST POINT SENSOR - pad PCB, bukan konektor tambahan"
Changed lines of the file:
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@@
 	(generator_version "10.0")
 	(paper "A4")
-	(text "K-16.2 | TEST POINT SENSOR - pad PCB, bukan konektor tambahan"
+	(text "TEST POINT SENSOR"
 		(exclude_from_sim no)
 		(at 30.48 22.86 0)

Commit message: Sync HAV and WBV KiCad sources with JLCPCB review packages
Parts:
- C4, C5: Assembly (none) -> JLCPCB Standard; Footprint_Status PROVISIONAL - package planning; not fabrication release -> ENGINEERING REVIEWED JLC-03; production release requires CA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; LCSC Part # (none) -> C3018562; Package 0805 / 2012 metric; X7R; 10% -> 100 nF; 50 V; X7R; 10%; 0805; Procurement_Status OPEN - exact MPN, datasheet and local stock must be verified -> FROZEN MPN JLC-02; selected for Standard PCBA; stock not re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; Supplier (none) -> JLCPCB; Supplier_URL (none) -> https://jlcpcb.com/partdetail/KEMET-C0805C104K5RACTU/C30185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
- C6: Assembly (none) -> JLCPCB Standard; Footprint_Status PROVISIONAL - package planning; not fabrication release -> ENGINEERING REVIEWED JLC-03; production release requires CA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; LCSC Part # (none) -> C2167376; Package 0805 / 2012 metric; X7R; 10% -> 1 uF; 16 V; X7R; 10%; 0805; Procurement_Status OPEN - exact MPN, datasheet and local stock must be verified -> FROZEN MPN JLC-02; selected for Standard PCBA; stock not re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; Supplier (none) -> JLCPCB; Supplier_URL (none) -> https://jlcpcb.com/partdetail/KEMET-C0805C105K4RACTU/C21673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
- R16: Assembly (none) -> JLCPCB Standard; Footprint_Status PROVISIONAL - package planning; not fabrication release -> ENGINEERING REVIEWED JLC-03; production release requires CA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; LCSC Part # (none) -> C96345; Package 0805 jumper; 0 ohm -> 0 ohm jumper; 0805; WAJIB terpasang, bukan DNP; Procurement_Status OPEN - exact MPN, datasheet and local stock must be verified -> FROZEN MPN JLC-02; selected for Standard PCBA; stock not re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; Supplier (none) -> JLCPCB; Supplier_URL (none) -> https://jlcpcb.com/partdetail/YAGEO-RC0805JR070RL/C96345
- R7: Assembly (none) -> JLCPCB Standard; Footprint_Status PROVISIONAL - package planning; not fabrication release -> ENGINEERING REVIEWED JLC-03; production release requires CA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; LCSC Part # (none) -> C84376; Package 0805 / 2012 metric; 1%; 0.125W -> 10 kohm; 1%; 0.125 W; 0805; Procurement_Status OPEN - exact MPN, datasheet and local stock must be verified -> FROZEN MPN JLC-02; selected for Standard PCBA; stock not re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; Supplier (none) -> JLCPCB; Supplier_URL (none) -> https://jlcpcb.com/partdetail/Yageo-RC0805FR0710KL/C84376
- U2: footprint ta_vibration_footprints:ADXL345_CC-14-1_Spectra_CANDIDATE -> hav_jlc:ADXL345_CC-14-1_ADI_JLC; Assembly (none) -> JLCPCB Standard; Footprint_Status PROVISIONAL ENGINEERING SELECTED 2026-09-28; pad gap 0.270m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 -> ENGINEERING REVIEWED JLC-03; production release requires CA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; LCSC Part # (none) -> C9667; Package CC-14-1; LGA-14; body 3x5mm; pitch 0.8mm -> Bare IC; LGA-14 CC-14-1; 3x5 mm; pitch 0.8 mm; Procurement_Status OPEN - verify genuine bare IC and local supplier; not a bre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 -> FROZEN MPN JLC-02; selected for Standard PCBA; stock not re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; Supplier (none) -> JLCPCB; Supplier_URL (none) -> https://jlcpcb.com/partdetail/AnalogDevices-ADXL345BCCZRL7/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
