File: hav_node/hav_connectors_testpoints.kicad_sch (KiCad schematic)
At the start: 7 parts, among them J3 KY016_EXTERNAL

Commit message: Rapihin skematik HAV
Other:
- note added: "KY-016 EKSTERNAL - J3"
- note removed: "Modul eksternal lewat J3, dikendalikan ESP32"
Changed lines of the file:
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@@
 	(title_block
 		(title "HAV - KY016 BATTERY INDICATOR")
-		(date "2026-09-08")
-		(rev "A0-RGB-DRAFT")
-		(comment 1 "PROVISIONAL - NOT FOR FABRICATION")
+		(date "2026-09-30")
+		(rev "A-CAM-REVIEW")
 	)
-	(text "Modul eksternal lewat J3, dikendalikan ESP32"
+	(text "KY-016 EKSTERNAL - J3"
 		(exclude_from_sim no)
 		(at 30.48 35.56 0)

Commit message: Sync HAV and WBV KiCad sources with JLCPCB review packages
Parts:
- J3: Assembly (none) -> JLCPCB Standard; Footprint_Status PROVISIONAL - selected geometry; exact purchased part verif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 -> ENGINEERING REVIEWED JLC-03; production release requires CA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; LCSC Part # (none) -> C144395; Package XH 4 pin vertical, 2.50mm pitch -> XH vertical 4 pin; pitch 2.50 mm; 3 A; Procurement_Status OPEN - indexed Shopee listing; stock, origin and exact vari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 -> FROZEN MPN JLC-02; selected for Standard PCBA; stock not re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; Supplier (none) -> JLCPCB; Supplier_URL https://shopee.co.id/Connector-XH-2.54-PCB-Male-2P-3P-4P-5P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 -> https://jlcpcb.com/partdetail/JST-B4B_XH_A_LF_SN/C144395
- R10, R11, R12: Assembly (none) -> JLCPCB Standard; Footprint_Status PROVISIONAL - package planning; not fabrication release -> ENGINEERING REVIEWED JLC-03; production release requires CA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; LCSC Part # (none) -> C114519; Package 0805 / 2012 metric; 1%; 0.125W -> 220 ohm; 1%; 0.125 W; 0805; Procurement_Status OPEN - exact MPN, datasheet and local stock must be verified -> FROZEN MPN JLC-02; selected for Standard PCBA; stock not re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; Supplier (none) -> JLCPCB; Supplier_URL (none) -> https://jlcpcb.com/partdetail/YAGEO-RC0805FR07220RL/C114519
- R13, R14, R15: Assembly (none) -> JLCPCB Standard; Footprint_Status PROVISIONAL - package planning; not fabrication release -> ENGINEERING REVIEWED JLC-03; production release requires CA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; LCSC Part # (none) -> C96346; Package 0805 / 2012 metric; 1%; 0.125W -> 100 kohm; 1%; 0.125 W; 0805; Procurement_Status OPEN - exact MPN, datasheet and local stock must be verified -> FROZEN MPN JLC-02; selected for Standard PCBA; stock not re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; Supplier (none) -> JLCPCB; Supplier_URL (none) -> https://jlcpcb.com/partdetail/YAGEO-RC0805FR07100KL/C96346
