File: hav_node/hav_esp32_programming.kicad_sch (KiCad schematic)
At the start: 17 parts, among them J1 PROG_UART, SW1 RESET, SW2 BOOT, U1 ESP32-WROOM-32E-N4

Commit message: Rapihin skematik HAV
Other:
- note added: "TEST POINT PROGRAMMING"
- note removed: "K-16.2 | TEST POINT PROGRAMMING"
Changed lines of the file:
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@@
 	(generator_version "10.0")
 	(paper "A4")
-	(text "K-16.2 | TEST POINT PROGRAMMING"
+	(text "TEST POINT PROGRAMMING"
 		(exclude_from_sim no)
 		(at 30.48 162.56 0)

Commit message: Sync HAV and WBV KiCad sources with JLCPCB review packages
Parts:
- C1: Assembly (none) -> JLCPCB Standard; Footprint_Status FROZEN geometry for selected MPN; assembly review required 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 -> ENGINEERING REVIEWED JLC-03; production release requires CA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; LCSC Part # (none) -> C90146; Package 1206 (3216 metric); 3.2x1.6x1.6mm nominal; X5R; 10%; 16V -> 22 uF; 16 V; X5R; 10%; 1206; Procurement_Status PROVISIONAL - Indonesian listing found; verify live stock, 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 -> FROZEN MPN JLC-02; selected for Standard PCBA; stock not re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; Supplier (none) -> JLCPCB; Supplier_URL https://shopee.co.id/product/9011098/20078115669 -> https://jlcpcb.com/partdetail/CL31A226KOHNNNE/C90146
- C2: Assembly (none) -> JLCPCB Standard; Footprint_Status PROVISIONAL - package planning; not fabrication release -> ENGINEERING REVIEWED JLC-03; production release requires CA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; LCSC Part # (none) -> C3018562; Package 0805 / 2012 metric; X7R; 10% -> 100 nF; 50 V; X7R; 10%; 0805; Procurement_Status OPEN - exact MPN, datasheet and local stock must be verified -> FROZEN MPN JLC-02; selected for Standard PCBA; stock not re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; Supplier (none) -> JLCPCB; Supplier_URL (none) -> https://jlcpcb.com/partdetail/KEMET-C0805C104K5RACTU/C30185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
- C3: Assembly (none) -> JLCPCB Standard; Footprint_Status PROVISIONAL - package planning; not fabrication release -> ENGINEERING REVIEWED JLC-03; production release requires CA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; LCSC Part # (none) -> C2167376; Package 0805 / 2012 metric; X7R; 10% -> 1 uF; 16 V; X7R; 10%; 0805; Procurement_Status OPEN - exact MPN, datasheet and local stock must be verified -> FROZEN MPN JLC-02; selected for Standard PCBA; stock not re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; Supplier (none) -> JLCPCB; Supplier_URL (none) -> https://jlcpcb.com/partdetail/KEMET-C0805C105K4RACTU/C21673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
- J1: footprint Connector_PinHeader_2.54mm:PinHeader_1x06_P2.54mm_Vertical -> Connector_HAV_JLC:PinHeader_1x06_P2.54mm_ZHOURI_1.02mm; Assembly (none) -> JLCPCB Standard; Footprint_Status PROVISIONAL - selected geometry; exact purchased part verif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 -> ENGINEERING REVIEWED JLC-03; production release requires CA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; LCSC Part # (none) -> C5156615; MPN OPEN - generic straight 1x06 2.54mm; manufacturer not discl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 -> 2.54-1*6; Manufacturer OPEN -> ZHOURI; Package THT straight male header, six positions, P2.54mm, square pi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 -> THT male 1x06 P2.54; pin 0.63mm square; drill 1.02mm; insul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; Procurement_Status OPEN - indexed Shopee listing; stock, origin and exact vari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 -> FROZEN MPN JLC-02; selected for Standard PCBA; stock not re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; Supplier (none) -> JLCPCB; Supplier_URL https://shopee.co.id/Breakable-Pin-Header-40-Pin-1x40-Male-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 -> https://jlcpcb.com/partdetail/ZHOURI-2_54_16/C5156615
- R1, R2: Assembly (none) -> JLCPCB Standard; Footprint_Status PROVISIONAL - package planning; not fabrication release -> ENGINEERING REVIEWED JLC-03; production release requires CA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; LCSC Part # (none) -> C84376; Package 0805 / 2012 metric; 1%; 0.125W -> 10 kohm; 1%; 0.125 W; 0805; Procurement_Status OPEN - exact MPN, datasheet and local stock must be verified -> FROZEN MPN JLC-02; selected for Standard PCBA; stock not re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; Supplier (none) -> JLCPCB; Supplier_URL (none) -> https://jlcpcb.com/partdetail/Yageo-RC0805FR0710KL/C84376
- R3: Assembly (none) -> JLCPCB Standard; Footprint_Status PROVISIONAL - package planning; not fabrication release -> ENGINEERING REVIEWED JLC-03; production release requires CA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; LCSC Part # (none) -> C130458; Package 0805 / 2012 metric; 1%; 0.125W -> 499 ohm; 1%; 0.125 W; 0805; Procurement_Status OPEN - exact MPN, datasheet and local stock must be verified -> FROZEN MPN JLC-02; selected for Standard PCBA; stock not re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; Supplier (none) -> JLCPCB; Supplier_URL (none) -> https://jlcpcb.com/partdetail/YAGEO-RC0805FR07499RL/C130458
- R4, R5, R6: Assembly (none) -> JLCPCB Standard; Footprint_Status PROVISIONAL - package planning; not fabrication release -> ENGINEERING REVIEWED JLC-03; production release requires CA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; LCSC Part # (none) -> C126353; Package 0805 / 2012 metric; 1%; 0.125W -> 33 ohm; 1%; 0.125 W; 0805; Procurement_Status OPEN - exact MPN, datasheet and local stock must be verified -> FROZEN MPN JLC-02; selected for Standard PCBA; stock not re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; Supplier (none) -> JLCPCB; Supplier_URL (none) -> https://jlcpcb.com/partdetail/YAGEO-RC0805FR0733RL/C126353
- SW1, SW2: Assembly (none) -> JLCPCB Standard; Footprint_Status FROZEN geometry for B3F-1000; receipt and authenticity veri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 -> ENGINEERING REVIEWED JLC-03; production release requires CA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; LCSC Part # (none) -> C93157; Package 6x6mm tactile NO, H4.3mm; holes 6.5x4.5mm -> Momentary SPST-NO; 6x6 mm; H4.3 mm; RESET / BOOT; Procurement_Status OPEN - indexed Shopee listing; stock, origin and exact vari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 -> FROZEN MPN JLC-02; selected for Standard PCBA; stock not re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; Supplier (none) -> JLCPCB; Supplier_URL https://shopee.co.id/Omron-B3F-1000-Mouse-Micro-Switch-Repl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 -> https://jlcpcb.com/partdetail/OmronElectronics-B3F1000/C931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
- U1: footprint ta_vibration_footprints:ESP32-WROOM-32E_NoThermalVias -> hav_jlc:ESP32-WROOM-32E_JLC_NoVia; Assembly (none) -> JLCPCB Standard; Footprint_Status PROVISIONAL - S02 no thermal PTH; preserve SMD EPAD; connec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 -> ENGINEERING REVIEWED JLC-03; production release requires CA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; LCSC Part # (none) -> C701341; Package (none) -> WROOM-32E; 4 MB flash; PCB antenna; bukan DevKit; Procurement_Status (none) -> FROZEN MPN JLC-02; selected for Standard PCBA; stock not re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; Supplier (none) -> JLCPCB; Supplier_URL (none) -> https://jlcpcb.com/partdetail/EspressifSystems-ESP32_WROOM_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
