File: hav_node/hav_node.kicad_pcb (KiCad board)
At the start: 2 copper layers, 56 x 36 mm, 54 parts, among them J1 PROG_UART, J2 BATTERY_2S_INPUT, J3 KY016_EXTERNAL, SW1 RESET, SW2 BOOT, SW3 KCD11-101 ON/OFF, U1 ESP32-WROOM-32E-N4, U2 ADXL345BCCZ-RL7, U3 MP1584 fixed 3V3 (PROV)

Commit message: HAV: final CAD check and cleanup 2026-10-02
Other:
- board text added: "CAM REVIEW - DFM / MECHANICAL FIT PENDING"
- board text removed: "CASING FIT / BATTERY UNVERIFIED - NO ROUTING"
Changed lines of the file:
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@@
 (gr_rect (start 100 78) (end 156 114) (stroke (width 0.05) (type default)) (fill none) (locked yes) (layer "Edge.Cuts"))
 (gr_text "PCB HAV 56 x 36 x 1.6 mm - RECTANGLE" (at 128 119) (layer "Dwgs.User") (effects (font (size 1 1) (thickness 0.15))))
-(gr_text "CASING FIT / BATTERY UNVERIFIED - NO ROUTING" (at 128 122) (layer "Dwgs.User") (effects (font (size 1 1) (thickness 0.15))))
+(gr_text "CAM REVIEW - DFM / MECHANICAL FIT PENDING" (at 128 122) (layer "Dwgs.User") (effects (font (size 1 1) (thickness 0.15))))
 (gr_text "U3 = WIRES TO EXTERNAL BUCK" (at 133 116) (layer "Dwgs.User") (effects (font (size 1 1) (thickness 0.15))))
 (gr_text "IN+" (at 126.5 109.25) (layer "F.SilkS") (effects (font (size 1 1) (thickness 0.21))))
@@
 (segment (start 144.7 96.45) (end 145.15 97.4) (width 0.5)(layer "F.Cu" )(net "3V3_SYS"))
 (net 49 "/HAV_ADXL345/GND_ADXL")
-(footprint "Resistor_SMD:R_0805_2012Metric"(layer "F.Cu" )(at 144.7 95.4 180)(descr "Resistor SMD 0805 (2012 Metric), square (rectangular) end terminal, IPC-7351 nominal, (Body size source: IPC-SM-782 page 72, https://www.pcb-3d.com/wordpress/wp-content/uploads/ipc-sm-782a_amendment_1_and_2.pdf)")(tags "resistor")(property "Reference" "R16"(at 0 -1.65 180)(layer "F.Fab" )(effects(font(size 1 1)(thickness 0.15))))(property "Value" "0R"(at 0 1.65 180)(layer "F.Fab" )(hide yes)(effects(font(size 1 1)(thickness 0.15))))(property "Datasheet" ""(at 0 0 180)(layer "F.Fab" )(hide yes)(effects(font(size 1.27 1.27))))(property "Description" ""(at 0 0 180)(layer "F.Fab" )(hide yes)(effects(font(size 1.27 1.27))))(property "KiLib_Generator" "SMD_2terminal_chip_molded"(at 0 0 180)(layer "F.SilkS" )(hide yes)(effects(font(size 1 1)(thickness 0.15))))(property "Datasheet" "https://www.yageogroup.com/component-documentation/download/specsheet/RC0805JR-070RL"(at 0 0 0)(layer "F.SilkS" )(hide yes)(effects(font(size 1.27 1.27))))(property "Description" "Resistor"(at 0 0 0)(layer "F.SilkS" )(hide yes)(effects(font(size 1.27 1.27))))(property "Package" "0805 jumper; 0 ohm"(at 0 0 0)(layer "F.SilkS" )(hide yes)(effects(font(size 1.27 1.27))))(property "Footprint_Status" "PROVISIONAL - package planning; not fabrication release"(at 0 0 0)(layer "F.SilkS" )(hide yes)(effects(font(size 1.27 1.27))))(property "MPN" "RC0805JR-070RL"(at 0 0 0)(layer "F.SilkS" )(hide yes)(effects(font(size 1.27 1.27))))(property "Procurement_Status" "OPEN - exact MPN, datasheet and local stock must be verified"(at 0 0 0)(layer "F.SilkS" )(hide yes)(effects(font(size 1.27 1.27))))(property "Manufacturer" "Yageo"(at 0 0 0)(layer "F.SilkS" )(hide yes)(effects(font(size 1.27 1.27))))(property "Design_Status" "FROZEN nominal/package; equivalent supplier part requires verification"(at 0 0 0)(layer "F.SilkS" )(hide yes)(effects(font(size 1.27 1.27))))(attr smd)(duplicate_pad_numbers_are_jumpers no)(fp_line (start -0.227064 0.735) (end 0.227064 0.735)(stroke (width 0.21) (type solid))(layer "F.SilkS" ))(fp_line (start -0.227064 -0.735) (end 0.227064 -0.735)(stroke (width 0.21) (type solid))(layer "F.SilkS" ))(fp_rect (start -1.68 -0.95) (end 1.68 0.95)(stroke (width 0.05) (type solid))(fill no)(layer "F.CrtYd" ))(fp_rect (start -1 -0.625) (end 1 0.625)(stroke (width 0.1) (type solid))(fill no)(layer "F.Fab" ))(fp_text user "${REFERENCE}"(at 0 0 180)(layer "F.Fab" )(effects(font(size 0.5 0.5)(thickness 0.08))))(pad "1" smd roundrect(at -0.9125 0 180)(size 1.025 1.4)(layers  "F.Cu" "F.Mask" "F.Paste")(roundrect_rratio 0.243902)(net "/HAV_ADXL345/GND_ADXL"))(pad "2" smd roundrect(at 0.9125 0 180)(size 1.025 1.4)(layers  "F.Cu" "F.Mask" "F.Paste")(roundrect_rratio 0.243902)(net "GND"))(embedded_fonts no)(model "${KICAD10_3DMODEL_DIR}/Resistor_SMD.3dshapes/R_0805_2012Metric.step"(offset (xyz 0 0 0))(scale (xyz 1 1 1))(rotate (xyz 0 0 0))))
+(footprint "Resistor_SMD:R_0805_2012Metric"(layer "F.Cu" )(at 144.7 95.4 180)(descr "Resistor SMD 0805 (2012 Metric), square (rectangular) end terminal, IPC-7351 nominal, (Body size source: IPC-SM-782 page 72, https://www.pcb-3d.com/wordpress/wp-content/uploads/ipc-sm-782a_amendment_1_and_2.pdf)")(tags "resistor")(property "Reference" "R16"(at 0 -1.65 180)(layer "F.Fab" )(effects(font(size 1 1)(thickness 0.15))))(property "Value" "0R"(at 0 1.65 180)(layer "F.Fab" )(hide yes)(effects(font(size 1 1)(thickness 0.15))))(property "KiLib_Generator" "SMD_2terminal_chip_molded"(at 0 0 180)(layer "F.SilkS" )(hide yes)(effects(font(size 1 1)(thickness 0.15))))(property "Datasheet" "https://www.yageogroup.com/component-documentation/download/specsheet/RC0805JR-070RL"(at 0 0 0)(layer "F.SilkS" )(hide yes)(effects(font(size 1.27 1.27))))(property "Description" "Resistor"(at 0 0 0)(layer "F.SilkS" )(hide yes)(effects(font(size 1.27 1.27))))(property "Package" "0805 jumper; 0 ohm"(at 0 0 0)(layer "F.SilkS" )(hide yes)(effects(font(size 1.27 1.27))))(property "Footprint_Status" "PROVISIONAL - package planning; not fabrication release"(at 0 0 0)(layer "F.SilkS" )(hide yes)(effects(font(size 1.27 1.27))))(property "MPN" "RC0805JR-070RL"(at 0 0 0)(layer "F.SilkS" )(hide yes)(effects(font(size 1.27 1.27))))(property "Procurement_Status" "OPEN - exact MPN, datasheet and local stock must be verified"(at 0 0 0)(layer "F.SilkS" )(hide yes)(effects(font(size 1.27 1.27))))(property "Manufacturer" "Yageo"(at 0 0 0)(layer "F.SilkS" )(hide yes)(effects(font(size 1.27 1.27))))(property "Design_Status" "FROZEN nominal/package; equivalent supplier part requires verification"(at 0 0 0)(layer "F.SilkS" )(hide yes)(effects(font(size 1.27 1.27))))(attr smd)(duplicate_pad_numbers_are_jumpers no)(fp_line (start -0.227064 0.735) (end 0.227064 0.735)(stroke (width 0.21) (type solid))(layer "F.SilkS" ))(fp_line (start -0.227064 -0.735) (end 0.227064 -0.735)(stroke (width 0.21) (type solid))(layer "F.SilkS" ))(fp_rect (start -1.68 -0.95) (end 1.68 0.95)(stroke (width 0.05) (type solid))(fill no)(layer "F.CrtYd" ))(fp_rect (start -1 -0.625) (end 1 0.625)(stroke (width 0.1) (type solid))(fill no)(layer "F.Fab" ))(fp_text user "${REFERENCE}"(at 0 0 180)(layer "F.Fab" )(effects(font(size 0.5 0.5)(thickness 0.08))))(pad "1" smd roundrect(at -0.9125 0 180)(size 1.025 1.4)(layers  "F.Cu" "F.Mask" "F.Paste")(roundrect_rratio 0.243902)(net "/HAV_ADXL345/GND_ADXL"))(pad "2" smd roundrect(at 0.9125 0 180)(size 1.025 1.4)(layers  "F.Cu" "F.Mask" "F.Paste")(roundrect_rratio 0.243902)(net "GND"))(embedded_fonts no)(model "${KICAD10_3DMODEL_DIR}/Resistor_SMD.3dshapes/R_0805_2012Metric.step"(offset (xyz 0 0 0))(scale (xyz 1 1 1))(rotate (xyz 0 0 0))))
 (segment (start 147.3025 95.4) (end 145.6125 95.4) (width 0.3)(layer "F.Cu" )(net "/HAV_ADXL345/GND_ADXL"))
 (segment (start 143.2338 93.0024) (end 148.3914 98.16) (width 0.3)(layer "B.Cu" )(net "/HAV_ESP32_PROGRAMMING/ESP_EN"))

Commit message: Sync HAV and WBV KiCad sources with JLCPCB review packages
Parts:
- J1: footprint Connector_PinHeader_2.54mm:PinHeader_1x06_P2.54mm_Vertical -> Connector_HAV_JLC:PinHeader_1x06_P2.54mm_ZHOURI_1.02mm
- U1: footprint ta_vibration_footprints:ESP32-WROOM-32E_NoThermalVias -> hav_jlc:ESP32-WROOM-32E_JLC_NoVia
- U2: footprint ta_vibration_footprints:ADXL345_CC-14-1_Spectra_CANDIDATE -> hav_jlc:ADXL345_CC-14-1_ADI_JLC
Other:
- rule pad_to_mask_clearance: 0.1016 -> 0.05
