File: hav_node/hav_power.kicad_sch (KiCad schematic)
At the start: 16 parts, among them J2 BATTERY_2S_INPUT, SW3 KCD11-101 ON/OFF, U3 MP1584 fixed 3V3 (PROV)

Commit message: Rapihin skematik HAV
Other:
- note added: "CATU DAYA HAV - LiPo 2S"
- note added: "PACK 2S BERPROTEKSI; CHARGING EKSTERNAL SAAT OFF. F1 BUKAN BMS; TP4056 TIDAK UNTUK 2S."
- note added: "PEMBACAAN BATERAI"
- note removed: "DRAFT / PROVISIONAL - Belum untuk produksi PCB"
- note removed: "K-15 | CATU DAYA HAV - LiPo 2S 1500 mAh"
- note removed: "K-15.8 | PEMBACAAN BATERAI"
- note removed: "OPEN: MPN, konektor/polaritas, BMS dan charger 2S. Pengisian eksternal: perangkat OFF; TP4056 tidak untuk 2S. F1 bukan pengganti BMS. 7.0 V belum menjadi cutoff final. REQ-PWR-01 >=8 jam; REQ-MEC-01/02 <=60x40x25 mm / 50 g."
- title: HAV POWER - K15 -> HAV POWER
Changed lines of the file:
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@@
 	(paper "A4")
 	(title_block
-		(title "HAV POWER - K15")
-		(date "2026-09-08")
-		(rev "A0-K15-DRAFT")
-		(comment 1 "PROVISIONAL - NOT FOR FABRICATION")
+		(title "HAV POWER")
+		(date "2026-09-30")
+		(rev "A-CAM-REVIEW")
 	)
-	(text "K-15 | CATU DAYA HAV - LiPo 2S 1500 mAh"
+	(text "CATU DAYA HAV - LiPo 2S"
 		(exclude_from_sim no)
 		(at 30.48 25.4 0)
@@
 		)
 	)
-	(text "K-15.8 | PEMBACAAN BATERAI"
+	(text "PEMBACAAN BATERAI"
 		(exclude_from_sim no)
 		(at 30.48 119.38 0)
@@
 		)
 	)
-	(text "OPEN: MPN, konektor/polaritas, BMS dan charger 2S.\nPengisian eksternal: perangkat OFF; TP4056 tidak untuk 2S.\nF1 bukan pengganti BMS. 7.0 V belum menjadi cutoff final.\nREQ-PWR-01 >=8 jam; REQ-MEC-01/02 <=60x40x25 mm / 50 g."
+	(text "PACK 2S BERPROTEKSI; CHARGING EKSTERNAL SAAT OFF.\nF1 BUKAN BMS; TP4056 TIDAK UNTUK 2S."
 		(exclude_from_sim no)
 		(at 30.48 182.88 0)
 		(effects
 			(font
-				(size 1.27 1.27)
-			)
-			(justify left top)
-		)
-	)
-	(text "DRAFT / PROVISIONAL - Belum untuk produksi PCB"
-		(exclude_from_sim no)
-		(at 30.48 33.02 0)
-		(effects
-			(font

Commit message: Sync HAV and WBV KiCad sources with JLCPCB review packages
Parts:
- C10, C11, C8: Assembly (none) -> JLCPCB Standard; Footprint_Status PROVISIONAL - package planning; not fabrication release -> ENGINEERING REVIEWED JLC-03; production release requires CA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; LCSC Part # (none) -> C3018562; Package 0805 / 2012 metric; X7R; 10% -> 100 nF; 50 V; X7R; 10%; 0805; Procurement_Status OPEN - exact MPN, datasheet and local stock must be verified -> FROZEN MPN JLC-02; selected for Standard PCBA; stock not re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; Supplier (none) -> JLCPCB; Supplier_URL (none) -> https://jlcpcb.com/partdetail/KEMET-C0805C104K5RACTU/C30185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
- C7, C9: Assembly (none) -> JLCPCB Standard; Footprint_Status FROZEN geometry for selected MPN; assembly review required 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 -> ENGINEERING REVIEWED JLC-03; production release requires CA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; LCSC Part # (none) -> C407893; Package Radial polar; D5mm x H11mm nominal; pitch 2mm; lead D0.5mm;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 -> 47 uF; 25 V; 20%; polar; radial D5 x H11 mm; pitch 2 mm; Procurement_Status PROVISIONAL - exact MPN listed on Monotaro Indonesia; Shope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 -> FROZEN MPN JLC-02; selected for Standard PCBA; stock not re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; Supplier (none) -> JLCPCB; Supplier_URL https://www.monotaro.id/s037414825.html -> https://jlcpcb.com/partdetail/PANASONIC-EEUFR1E470/C407893
- F1: Assembly (none) -> JLCPCB Standard; Footprint_Status PROVISIONAL - selected geometry; exact purchased part verif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 -> ENGINEERING REVIEWED JLC-03; production release requires CA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; LCSC Part # (none) -> C84140; Package 1812 Style1 PPTC; 0.75A hold, 1.5A trip at 23C; 13.2V max; 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 -> PTC; hold 0.75 A; trip 1.5 A; max 13.2 V; 1812 Style 1; Procurement_Status OPEN - indexed Shopee listing; stock, origin and exact vari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 -> FROZEN MPN JLC-02; selected for Standard PCBA; stock not re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; Supplier (none) -> JLCPCB; Supplier_URL https://shopee.co.id/SMD-PPTC-1812-0.75A-Self-Recovery-Fuse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 -> https://jlcpcb.com/partdetail/BOURNS-MF_MSMF0752/C84140
- J2: Assembly (none) -> JLCPCB Standard; Footprint_Status PROVISIONAL - selected geometry; exact purchased part verif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 -> ENGINEERING REVIEWED JLC-03; production release requires CA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; LCSC Part # (none) -> C158012; Package XH 2 pin vertical, 2.50mm pitch -> XH vertical 2 pin; pitch 2.50 mm; 3 A; Procurement_Status OPEN - indexed Shopee listing; stock, origin and exact vari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 -> FROZEN MPN JLC-02; selected for Standard PCBA; stock not re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; Supplier (none) -> JLCPCB; Supplier_URL https://shopee.co.id/Connector-XH-2.54-PCB-Male-2P-3P-4P-5P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 -> https://jlcpcb.com/partdetail/B2B-XH-A%28LF%29%28SN%29/C158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
- R8: Assembly (none) -> JLCPCB Standard; Footprint_Status PROVISIONAL - package planning; not fabrication release -> ENGINEERING REVIEWED JLC-03; production release requires CA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; LCSC Part # (none) -> C114528; Package 0805 / 2012 metric; 1%; 0.125W -> 330 kohm; 1%; 0.125 W; 0805; Procurement_Status OPEN - exact MPN, datasheet and local stock must be verified -> FROZEN MPN JLC-02; selected for Standard PCBA; stock not re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; Supplier (none) -> JLCPCB; Supplier_URL (none) -> https://jlcpcb.com/partdetail/YAGEO-RC0805FR07330KL/C114528
- R9: Assembly (none) -> JLCPCB Standard; Footprint_Status PROVISIONAL - package planning; not fabrication release -> ENGINEERING REVIEWED JLC-03; production release requires CA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; LCSC Part # (none) -> C96346; Package 0805 / 2012 metric; 1%; 0.125W -> 100 kohm; 1%; 0.125 W; 0805; Procurement_Status OPEN - exact MPN, datasheet and local stock must be verified -> FROZEN MPN JLC-02; selected for Standard PCBA; stock not re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; Supplier (none) -> JLCPCB; Supplier_URL (none) -> https://jlcpcb.com/partdetail/YAGEO-RC0805FR07100KL/C96346
