File: main_unit/main_adxl345.kicad_sch (KiCad schematic)
At the start: 11 parts, among them U2 ADXL345BCCZ-RL7

Commit message: Sync HAV and WBV KiCad sources with JLCPCB review packages
Parts:
- C4, C5: Assembly (none) -> JLCPCB Standard planned; process review pending; Footprint_Status (none) -> Layout baseline reviewed; final PCB DRC/DFM and assembly re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; LCSC Part # (none) -> C3018562; Manufacturer (none) -> KEMET; Procurement_Status PROVISIONAL - listing/candidate only; exact MPN and domesti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 -> FROZEN MPN/catalog identity; stock not reserved; order revi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; Selection_Note Sama dengan basis komponen HAV; tidak mengubah HAV. -> MPN dan footprint dipertahankan; baseline layout JLC, bukan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; Status FROZEN geometry; procurement PROVISIONAL -> FROZEN layout baseline; not production release; Supplier (none) -> JLCPCB; Supplier_URL https://shopee.co.id/product/25936178/8912815073 -> https://jlcpcb.com/partdetail/KEMET-C0805C104K5RACTU/C30185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
- C6: Assembly (none) -> JLCPCB Standard planned; process review pending; Footprint_Status (none) -> Layout baseline reviewed; final PCB DRC/DFM and assembly re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; LCSC Part # (none) -> C2167376; Manufacturer (none) -> KEMET; Procurement_Status PROVISIONAL - listing/candidate only; exact MPN and domesti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 -> FROZEN MPN/catalog identity; stock not reserved; order revi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; Selection_Note Sama dengan basis komponen HAV; tidak mengubah HAV. -> MPN dan footprint dipertahankan; baseline layout JLC, bukan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; Status FROZEN geometry; procurement PROVISIONAL -> FROZEN layout baseline; not production release; Supplier (none) -> JLCPCB; Supplier_URL https://shopee.co.id/product/25936178/24826003791 -> https://jlcpcb.com/partdetail/KEMET-C0805C105K4RACTU/C21673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
- FB1: Assembly (none) -> JLCPCB Standard planned; process review pending; Footprint_Status (none) -> Layout baseline reviewed; final PCB DRC/DFM and assembly re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; LCSC Part # (none) -> C41556732; Manufacturer (none) -> Murata Electronics; Procurement_Status PROVISIONAL - listing/candidate only; exact MPN and domesti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 -> FROZEN MPN/catalog identity; stock not reserved; order revi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; Selection_Note Bead Main tetap, tidak otomatis dihapus mengikuti HAV. Basi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 -> Bead WBV dipertahankan; berbeda dengan penghapusan bead HAV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; Status PROVISIONAL procurement; footprint selected -> FROZEN layout baseline; not production release; Supplier (none) -> JLCPCB; Supplier_URL https://shopee.co.id/search?keyword=BLM21PG601SN1D -> https://jlcpcb.com/partdetail/MurataElectronics-BLM21PG601S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
- U2: footprint ta_vibration_footprints:ADXL345_CC-14-1_Spectra_CANDIDATE -> wbv_jlc:ADXL345_CC-14-1_ADI_JLC; Assembly (none) -> JLCPCB Standard planned; process review pending; Footprint_Status (none) -> Layout baseline reviewed; final PCB DRC/DFM and assembly re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; LCSC Part # (none) -> C9667; Manufacturer (none) -> Analog Devices; Procurement_Status PROVISIONAL - listing/candidate only; exact MPN and domesti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 -> FROZEN MPN/catalog identity; stock not reserved; order revi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; Selection_Note Sama kandidat Spectra HAV; modified pad gap0.270mm. NOT off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 -> Land ADI 1.145x0.55mm, pitch0.8mm; menggantikan Spectra can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; Status PROVISIONAL Spectra candidate; fabrication approval BLOCKING -> FROZEN layout baseline; not production release; Supplier (none) -> JLCPCB; Supplier_URL https://shopee.co.id/search?keyword=ADXL345BCCZ%20IC%20LGA -> https://jlcpcb.com/partdetail/AnalogDevices-ADXL345BCCZRL7/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
