File: main_unit/main_coordinates.kicad_sch (KiCad schematic)
At the start: 6 parts, among them J5 GPS_UART_3V3

Commit message: Sync HAV and WBV KiCad sources with JLCPCB review packages
Parts:
- C23: Assembly (none) -> JLCPCB Standard planned; process review pending; Footprint_Status (none) -> Layout baseline reviewed; final PCB DRC/DFM and assembly re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; LCSC Part # (none) -> C15850; Manufacturer (none) -> Samsung Electro-Mechanics; Procurement_Status PROVISIONAL - listing/candidate only; exact MPN and domesti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 -> FROZEN MPN/catalog identity; stock not reserved; order revi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; Selection_Note Samsung resmi: 2.0x1.25x1.25mm; cek effective C. Listing te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 -> MPN dan footprint dipertahankan; baseline layout JLC, bukan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; Status FROZEN geometry; procurement PROVISIONAL -> FROZEN layout baseline; not production release; Supplier (none) -> JLCPCB; Supplier_URL https://shopee.co.id/product/45119540/7441919037 -> https://jlcpcb.com/partdetail/CL21A106KAYNNNE/C15850
- C24: Assembly (none) -> JLCPCB Standard planned; process review pending; Footprint_Status (none) -> Layout baseline reviewed; final PCB DRC/DFM and assembly re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; LCSC Part # (none) -> C3018562; Manufacturer (none) -> KEMET; Procurement_Status PROVISIONAL - listing/candidate only; exact MPN and domesti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 -> FROZEN MPN/catalog identity; stock not reserved; order revi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; Selection_Note Sama dengan basis komponen HAV; tidak mengubah HAV. -> MPN dan footprint dipertahankan; baseline layout JLC, bukan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; Status FROZEN geometry; procurement PROVISIONAL -> FROZEN layout baseline; not production release; Supplier (none) -> JLCPCB; Supplier_URL https://shopee.co.id/product/25936178/8912815073 -> https://jlcpcb.com/partdetail/KEMET-C0805C104K5RACTU/C30185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
- J5: Assembly (none) -> JLCPCB Standard planned; process review pending; Footprint_Status (none) -> Layout baseline reviewed; final PCB DRC/DFM and assembly re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; LCSC Part # (none) -> C144395; Manufacturer (none) -> JST; Procurement_Status PROVISIONAL - listing/candidate only; exact MPN and domesti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 -> FROZEN MPN/catalog identity; stock not reserved; order revi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; Selection_Note Konektor kabel sisi PCB, bukan footprint board OLED/GPS. Wa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 -> MPN dan footprint dipertahankan; baseline layout JLC, bukan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; Status FROZEN geometry; procurement PROVISIONAL -> FROZEN layout baseline; not production release; Supplier (none) -> JLCPCB; Supplier_URL https://shopee.co.id/Connector-XH-2.54-PCB-Male-2P-3P-4P-5P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 -> https://jlcpcb.com/partdetail/JST-B4B_XH_A_LF_SN/C144395
