File: main_unit/main_esp32_programming.kicad_sch (KiCad schematic)
At the start: 9 parts, among them SW1 RESET, SW2 BOOT, U1 ESP32-WROOM-32E-N4

Commit message: Sync HAV and WBV KiCad sources with JLCPCB review packages
Parts:
- C1: Assembly (none) -> JLCPCB Standard planned; process review pending; Footprint_Status (none) -> Layout baseline reviewed; final PCB DRC/DFM and assembly re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; LCSC Part # (none) -> C90146; Manufacturer (none) -> Samsung Electro-Mechanics; Procurement_Status PROVISIONAL - listing/candidate only; exact MPN and domesti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 -> FROZEN MPN/catalog identity; stock not reserved; order revi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; Selection_Note Sama dengan basis komponen HAV; tidak mengubah HAV. -> MPN dan footprint dipertahankan; baseline layout JLC, bukan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; Status FROZEN geometry; procurement PROVISIONAL -> FROZEN layout baseline; not production release; Supplier (none) -> JLCPCB; Supplier_URL https://shopee.co.id/product/9011098/20078115669 -> https://jlcpcb.com/partdetail/CL31A226KOHNNNE/C90146
- C2: Assembly (none) -> JLCPCB Standard planned; process review pending; Footprint_Status (none) -> Layout baseline reviewed; final PCB DRC/DFM and assembly re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; LCSC Part # (none) -> C3018562; Manufacturer (none) -> KEMET; Procurement_Status PROVISIONAL - listing/candidate only; exact MPN and domesti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 -> FROZEN MPN/catalog identity; stock not reserved; order revi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; Selection_Note Sama dengan basis komponen HAV; tidak mengubah HAV. -> MPN dan footprint dipertahankan; baseline layout JLC, bukan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; Status FROZEN geometry; procurement PROVISIONAL -> FROZEN layout baseline; not production release; Supplier (none) -> JLCPCB; Supplier_URL https://shopee.co.id/product/25936178/8912815073 -> https://jlcpcb.com/partdetail/KEMET-C0805C104K5RACTU/C30185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
- C3: Assembly (none) -> JLCPCB Standard planned; process review pending; Footprint_Status (none) -> Layout baseline reviewed; final PCB DRC/DFM and assembly re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; LCSC Part # (none) -> C2167376; Manufacturer (none) -> KEMET; Procurement_Status PROVISIONAL - listing/candidate only; exact MPN and domesti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 -> FROZEN MPN/catalog identity; stock not reserved; order revi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; Selection_Note Sama dengan basis komponen HAV; tidak mengubah HAV. -> MPN dan footprint dipertahankan; baseline layout JLC, bukan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; Status FROZEN geometry; procurement PROVISIONAL -> FROZEN layout baseline; not production release; Supplier (none) -> JLCPCB; Supplier_URL https://shopee.co.id/product/25936178/24826003791 -> https://jlcpcb.com/partdetail/KEMET-C0805C105K4RACTU/C21673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
- R1, R2: Assembly (none) -> JLCPCB Standard planned; process review pending; Footprint_Status (none) -> Layout baseline reviewed; final PCB DRC/DFM and assembly re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; LCSC Part # (none) -> C84376; Manufacturer (none) -> Yageo; Procurement_Status PROVISIONAL - listing/candidate only; exact MPN and domesti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 -> FROZEN MPN/catalog identity; stock not reserved; order revi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; Selection_Note Sama dengan basis komponen HAV; tidak mengubah HAV. -> MPN dan footprint dipertahankan; baseline layout JLC, bukan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; Status FROZEN geometry; procurement PROVISIONAL -> FROZEN layout baseline; not production release; Supplier (none) -> JLCPCB; Supplier_URL https://shopee.co.id/product/16973105/49051878593 -> https://jlcpcb.com/partdetail/Yageo-RC0805FR0710KL/C84376
- R3: Assembly (none) -> JLCPCB Standard planned; process review pending; Footprint_Status (none) -> Layout baseline reviewed; final PCB DRC/DFM and assembly re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; LCSC Part # (none) -> C130458; Manufacturer (none) -> Yageo; Procurement_Status PROVISIONAL - listing/candidate only; exact MPN and domesti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 -> FROZEN MPN/catalog identity; stock not reserved; order revi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; Selection_Note Sama dengan basis komponen HAV; tidak mengubah HAV. -> MPN dan footprint dipertahankan; baseline layout JLC, bukan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; Status FROZEN geometry; procurement PROVISIONAL -> FROZEN layout baseline; not production release; Supplier (none) -> JLCPCB; Supplier_URL https://shopee.co.id/search?keyword=resistor%200805%20499%2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 -> https://jlcpcb.com/partdetail/YAGEO-RC0805FR07499RL/C130458
- SW1, SW2: Assembly (none) -> JLCPCB Standard planned; process review pending; Footprint_Status (none) -> Layout baseline reviewed; final PCB DRC/DFM and assembly re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; LCSC Part # (none) -> C93157; MPN Generik OPEN; B3F-1000 hanya acuan drawing -> B3F-1000; Manufacturer (none) -> Omron; Package THT tactile NO 6x6mm H4.3mm; holes6.5x4.5mm -> Omron B3F-1000 THT tactile NO 6x6mm H4.3mm; terminal center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; Procurement_Status PROVISIONAL - listing/candidate only; exact MPN and domesti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 -> FROZEN MPN/catalog identity; stock not reserved; order revi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; Selection_Note Generik Aladin Shop varian4.3mm. Omron B3F1000 hanya refere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 -> Exact Omron B3F-1000 untuk PCBA menggantikan generic procur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; Status PROVISIONAL generic part; reference geometry selected -> FROZEN layout baseline; not production release; Supplier (none) -> JLCPCB; Supplier_URL https://shopee.co.id/product/7849796/24862806415 -> https://jlcpcb.com/partdetail/OmronElectronics-B3F1000/C931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
- U1: footprint ta_vibration_footprints:ESP32-WROOM-32E_NoThermalVias -> wbv_jlc:ESP32-WROOM-32E_JLC_NoVia; Assembly (none) -> JLCPCB Standard planned; process review pending; Footprint_Status (none) -> Layout baseline reviewed; final PCB DRC/DFM and assembly re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; LCSC Part # (none) -> C701341; Manufacturer (none) -> Espressif; Procurement_Status PROVISIONAL - listing/candidate only; exact MPN and domesti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 -> FROZEN MPN/catalog identity; stock not reserved; order revi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; Selection_Note Sama HAV no-thermal-via variant: all SMD pads/antenna keepo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 -> Varian Espressif reviewed dari HAV JLC-03; EPAD SMD dan ant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; Status PROVISIONAL engineering footprint; manufacturer land patter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 -> FROZEN layout baseline; not production release; Supplier (none) -> JLCPCB; Supplier_URL https://shopee.co.id/product/65450634/13839165245 -> https://jlcpcb.com/partdetail/EspressifSystems-ESP32_WROOM_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
