File: main_unit/main_hmi.kicad_sch (KiCad schematic)
At the start: 8 parts, among them SW3 START_STOP

Commit message: Sync HAV and WBV KiCad sources with JLCPCB review packages
Parts:
- C16, C22: Assembly (none) -> JLCPCB Standard planned; process review pending; Footprint_Status (none) -> Layout baseline reviewed; final PCB DRC/DFM and assembly re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; LCSC Part # (none) -> C3018562; Manufacturer (none) -> KEMET; Procurement_Status PROVISIONAL - listing/candidate only; exact MPN and domesti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 -> FROZEN MPN/catalog identity; stock not reserved; order revi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; Selection_Note Sama dengan basis komponen HAV; tidak mengubah HAV. -> MPN dan footprint dipertahankan; baseline layout JLC, bukan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; Status FROZEN geometry; procurement PROVISIONAL -> FROZEN layout baseline; not production release; Supplier (none) -> JLCPCB; Supplier_URL https://shopee.co.id/product/25936178/8912815073 -> https://jlcpcb.com/partdetail/KEMET-C0805C104K5RACTU/C30185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
- D3: footprint Package_TO_SOT_SMD:SOT-23-6 -> wbv_jlc:SOT-23-6_USBLC6-4SC6_ST; Assembly (none) -> JLCPCB Standard planned; process review pending; Footprint_Status (none) -> Layout baseline reviewed; final PCB DRC/DFM and assembly re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; LCSC Part # (none) -> C111212; Manufacturer (none) -> STMicroelectronics; Package SOT23-6; 4 data lines -> SOT23-6L; 4 data lines; ST Fig20 land pattern; Procurement_Status PROVISIONAL - listing/candidate only; exact MPN and domesti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 -> FROZEN MPN/catalog identity; stock not reserved; order revi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; Selection_Note Exact source Indonesia belum ditemukan. USBLC6-2SC6 lokal B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 -> Tetap USBLC6-4SC6; bukan 2SC6. Land resmi ST 1.2x0.6mm, pit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; Status PROVISIONAL procurement BLOCKING; retain existing 4SC6 circ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 -> FROZEN layout baseline; not production release; Supplier (none) -> JLCPCB; Supplier_URL https://shopee.co.id/search?keyword=USBLC6-4SC6 -> https://jlcpcb.com/partdetail/USBLC6-4SC6/C111212
- R19: Assembly (none) -> JLCPCB Standard planned; process review pending; Footprint_Status (none) -> Layout baseline reviewed; final PCB DRC/DFM and assembly re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; LCSC Part # (none) -> C84376; Manufacturer (none) -> Yageo; Procurement_Status PROVISIONAL - listing/candidate only; exact MPN and domesti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 -> FROZEN MPN/catalog identity; stock not reserved; order revi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; Selection_Note Sama dengan basis komponen HAV; tidak mengubah HAV. -> MPN dan footprint dipertahankan; baseline layout JLC, bukan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; Status FROZEN geometry; procurement PROVISIONAL -> FROZEN layout baseline; not production release; Supplier (none) -> JLCPCB; Supplier_URL https://shopee.co.id/product/16973105/49051878593 -> https://jlcpcb.com/partdetail/Yageo-RC0805FR0710KL/C84376
- R20: Assembly (none) -> JLCPCB Standard planned; process review pending; Footprint_Status (none) -> Layout baseline reviewed; final PCB DRC/DFM and assembly re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; LCSC Part # (none) -> C95781; Manufacturer (none) -> Yageo; Procurement_Status PROVISIONAL - listing/candidate only; exact MPN and domesti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 -> FROZEN MPN/catalog identity; stock not reserved; order revi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; Selection_Note Pilih varian nilai tepat; resistor generik bukan otomatis e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 -> MPN dan footprint dipertahankan; baseline layout JLC, bukan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; Status FROZEN geometry; procurement PROVISIONAL -> FROZEN layout baseline; not production release; Supplier (none) -> JLCPCB; Supplier_URL https://shopee.co.id/product/16973105/49051878593 -> https://jlcpcb.com/partdetail/YAGEO-RC0805FR071KL/C95781
- SW3: Assembly (none) -> JLCPCB Standard planned; process review pending; Footprint_Status (none) -> Layout baseline reviewed; final PCB DRC/DFM and assembly re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; LCSC Part # (none) -> C93157; MPN Generik OPEN; B3F-1000 hanya acuan drawing -> B3F-1000; Manufacturer (none) -> Omron; Package THT tactile NO 6x6mm H4.3mm; holes6.5x4.5mm -> Omron B3F-1000 THT tactile NO 6x6mm H4.3mm; terminal center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; Procurement_Status PROVISIONAL - listing/candidate only; exact MPN and domesti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 -> FROZEN MPN/catalog identity; stock not reserved; order revi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; Selection_Note Generik Aladin Shop varian4.3mm. Omron B3F1000 hanya refere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 -> Exact Omron B3F-1000 untuk PCBA menggantikan generic procur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; Status PROVISIONAL generic part; reference geometry selected -> FROZEN layout baseline; not production release; Supplier (none) -> JLCPCB; Supplier_URL https://shopee.co.id/product/7849796/24862806415 -> https://jlcpcb.com/partdetail/OmronElectronics-B3F1000/C931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
