File: main_unit/main_microsd.kicad_sch (KiCad schematic)
At the start: 23 parts, among them J2 DM3CS-SF

Commit message: Sync HAV and WBV KiCad sources with JLCPCB review packages
Parts:
- C10, C11, C12, C7: Assembly (none) -> JLCPCB Standard planned; process review pending; Footprint_Status (none) -> Layout baseline reviewed; final PCB DRC/DFM and assembly re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; LCSC Part # (none) -> C3018562; Manufacturer (none) -> KEMET; Procurement_Status PROVISIONAL - listing/candidate only; exact MPN and domesti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 -> FROZEN MPN/catalog identity; stock not reserved; order revi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; Selection_Note Sama dengan basis komponen HAV; tidak mengubah HAV. -> MPN dan footprint dipertahankan; baseline layout JLC, bukan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; Status FROZEN geometry; procurement PROVISIONAL -> FROZEN layout baseline; not production release; Supplier (none) -> JLCPCB; Supplier_URL https://shopee.co.id/product/25936178/8912815073 -> https://jlcpcb.com/partdetail/KEMET-C0805C104K5RACTU/C30185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
- C8: Assembly (none) -> JLCPCB Standard planned; process review pending; Footprint_Status (none) -> Layout baseline reviewed; final PCB DRC/DFM and assembly re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; LCSC Part # (none) -> C15850; Manufacturer (none) -> Samsung Electro-Mechanics; Procurement_Status PROVISIONAL - listing/candidate only; exact MPN and domesti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 -> FROZEN MPN/catalog identity; stock not reserved; order revi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; Selection_Note Samsung resmi: 2.0x1.25x1.25mm; cek effective C. Listing te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 -> MPN dan footprint dipertahankan; baseline layout JLC, bukan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; Status FROZEN geometry; procurement PROVISIONAL -> FROZEN layout baseline; not production release; Supplier (none) -> JLCPCB; Supplier_URL https://shopee.co.id/product/45119540/7441919037 -> https://jlcpcb.com/partdetail/CL21A106KAYNNNE/C15850
- D1, D2: footprint Package_TO_SOT_SMD:SOT-23-6 -> wbv_jlc:SOT-23-6_USBLC6-4SC6_ST; Assembly (none) -> JLCPCB Standard planned; process review pending; Footprint_Status (none) -> Layout baseline reviewed; final PCB DRC/DFM and assembly re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; LCSC Part # (none) -> C111212; Manufacturer (none) -> STMicroelectronics; Package SOT23-6; 4 data lines -> SOT23-6L; 4 data lines; ST Fig20 land pattern; Procurement_Status PROVISIONAL - listing/candidate only; exact MPN and domesti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 -> FROZEN MPN/catalog identity; stock not reserved; order revi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; Selection_Note Exact source Indonesia belum ditemukan. USBLC6-2SC6 lokal B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 -> Tetap USBLC6-4SC6; bukan 2SC6. Land resmi ST 1.2x0.6mm, pit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; Status PROVISIONAL procurement BLOCKING; retain existing 4SC6 circ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 -> FROZEN layout baseline; not production release; Supplier (none) -> JLCPCB; Supplier_URL https://shopee.co.id/search?keyword=USBLC6-4SC6 -> https://jlcpcb.com/partdetail/USBLC6-4SC6/C111212
- J2: footprint (none) -> wbv_jlc:microSD_Hirose_DM3CS-SF; Assembly (none) -> JLCPCB SMT assembly planned; holder/socket only; Footprint_Status (none) -> Manufacturer drawing reviewed; final placement DRC/DFM/CPL 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; LCSC Part # (none) -> C202111; Manufacturer (none) -> Hirose Electric; Package (none) -> SMT hinged microSD 13.8x14.1mm H1.83mm; card detect + four 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; Procurement_Status (none) -> FROZEN exact MPN/C-code; stock snapshot2026-10-06 not reser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; Selection_Note (none) -> Manufacturer p7 confirms CD closes to shell/GND with card i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; Status PROVISIONAL - not for fabrication -> FROZEN layout baseline; not production release; Supplier (none) -> JLCPCB; Supplier_URL (none) -> https://jlcpcb.com/partdetail/hrs_hirose-DM3CSSF/C202111
- R10, R8, R9: Assembly (none) -> JLCPCB Standard planned; process review pending; Footprint_Status (none) -> Layout baseline reviewed; final PCB DRC/DFM and assembly re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; LCSC Part # (none) -> C126353; Manufacturer (none) -> Yageo; Procurement_Status PROVISIONAL - listing/candidate only; exact MPN and domesti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 -> FROZEN MPN/catalog identity; stock not reserved; order revi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; Selection_Note Sama dengan basis komponen HAV; tidak mengubah HAV. -> MPN dan footprint dipertahankan; baseline layout JLC, bukan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; Status FROZEN geometry; procurement PROVISIONAL -> FROZEN layout baseline; not production release; Supplier (none) -> JLCPCB; Supplier_URL https://shopee.co.id/search?keyword=resistor%200805%2033%20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 -> https://jlcpcb.com/partdetail/YAGEO-RC0805FR0733RL/C126353
- R11, R12, R13, R14, R15, R16: Assembly (none) -> JLCPCB Standard planned; process review pending; Footprint_Status (none) -> Layout baseline reviewed; final PCB DRC/DFM and assembly re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; LCSC Part # (none) -> C84376; Manufacturer (none) -> Yageo; Procurement_Status PROVISIONAL - listing/candidate only; exact MPN and domesti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 -> FROZEN MPN/catalog identity; stock not reserved; order revi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; Selection_Note Sama dengan basis komponen HAV; tidak mengubah HAV. -> MPN dan footprint dipertahankan; baseline layout JLC, bukan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; Status FROZEN geometry; procurement PROVISIONAL -> FROZEN layout baseline; not production release; Supplier (none) -> JLCPCB; Supplier_URL https://shopee.co.id/product/16973105/49051878593 -> https://jlcpcb.com/partdetail/Yageo-RC0805FR0710KL/C84376
Other:
- note added: "J2: DM3CS-SF | hinged | card detect"
- note removed: "J2: HOLD - pilihan soket menunggu tim"
