File: main_unit/main_power.kicad_sch (KiCad schematic)
At the start: 16 parts, among them J4 PACK_2S_P+/P-, SW4 POWER_ON_OFF, U4 MP1584 MODULE 3V3 (PROV)

Commit message: Sync HAV and WBV KiCad sources with JLCPCB review packages
Parts:
- C17, C19: Assembly (none) -> JLCPCB Standard planned; process review pending; Footprint_Status (none) -> Layout baseline reviewed; final PCB DRC/DFM and assembly re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; LCSC Part # (none) -> C407893; Manufacturer (none) -> Panasonic; Procurement_Status PROVISIONAL - listing/candidate only; exact MPN and domesti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 -> FROZEN MPN/catalog identity; stock not reserved; order revi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; Selection_Note Sama dengan basis komponen HAV; tidak mengubah HAV. -> MPN dan footprint dipertahankan; baseline layout JLC, bukan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; Status FROZEN geometry; procurement PROVISIONAL -> FROZEN layout baseline; not production release; Supplier (none) -> JLCPCB; Supplier_URL https://www.monotaro.id/s037414825.html -> https://jlcpcb.com/partdetail/PANASONIC-EEUFR1E470/C407893
- C18, C20, C21: Assembly (none) -> JLCPCB Standard planned; process review pending; Footprint_Status (none) -> Layout baseline reviewed; final PCB DRC/DFM and assembly re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; LCSC Part # (none) -> C3018562; Manufacturer (none) -> KEMET; Procurement_Status PROVISIONAL - listing/candidate only; exact MPN and domesti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 -> FROZEN MPN/catalog identity; stock not reserved; order revi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; Selection_Note Sama dengan basis komponen HAV; tidak mengubah HAV. -> MPN dan footprint dipertahankan; baseline layout JLC, bukan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; Status FROZEN geometry; procurement PROVISIONAL -> FROZEN layout baseline; not production release; Supplier (none) -> JLCPCB; Supplier_URL https://shopee.co.id/product/25936178/8912815073 -> https://jlcpcb.com/partdetail/KEMET-C0805C104K5RACTU/C30185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
- F1: Assembly (none) -> JLCPCB Standard planned; process review pending; Footprint_Status (none) -> Layout baseline reviewed; final PCB DRC/DFM and assembly re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; LCSC Part # (none) -> C84140; Manufacturer (none) -> Bourns; Procurement_Status PROVISIONAL - listing/candidate only; exact MPN and domesti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 -> FROZEN MPN/catalog identity; stock not reserved; order revi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; Selection_Note WBV-04: retain 0.75A input PTC provisionally; hot derating/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 -> Exact MF-MSMF075-2; rating0.75A tetap PROVISIONAL terhadap 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; Status PROVISIONAL rating and procurement; footprint selected -> FROZEN MPN/footprint; PROVISIONAL rating derating/inrush ve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; Supplier (none) -> JLCPCB; Supplier_URL https://shopee.co.id/search?keyword=MF%20MSMF075%202%201812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 -> https://jlcpcb.com/partdetail/BOURNS-MF_MSMF0752/C84140
- J4: Assembly (none) -> JLCPCB Standard planned; process review pending; Footprint_Status (none) -> Layout baseline reviewed; final PCB DRC/DFM and assembly re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; LCSC Part # (none) -> C158012; Manufacturer (none) -> JST; Procurement_Status PROVISIONAL - listing/candidate only; exact MPN and domesti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 -> FROZEN MPN/catalog identity; stock not reserved; order revi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; Selection_Note Sama HAV J2; pin1=P+ protected, pin2=P-. Generic 2.54mm tid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 -> MPN dan footprint dipertahankan; baseline layout JLC, bukan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; Status FROZEN geometry; procurement PROVISIONAL -> FROZEN layout baseline; not production release; Supplier (none) -> JLCPCB; Supplier_URL https://shopee.co.id/Connector-XH-2.54-PCB-Male-2P-3P-4P-5P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 -> https://jlcpcb.com/partdetail/B2B-XH-A%28LF%29%28SN%29/C158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
- R21: Assembly (none) -> JLCPCB Standard planned; process review pending; Footprint_Status (none) -> Layout baseline reviewed; final PCB DRC/DFM and assembly re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; LCSC Part # (none) -> C114528; Manufacturer (none) -> Yageo; Procurement_Status PROVISIONAL - listing/candidate only; exact MPN and domesti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 -> FROZEN MPN/catalog identity; stock not reserved; order revi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; Selection_Note Sama dengan basis komponen HAV; tidak mengubah HAV. -> MPN dan footprint dipertahankan; baseline layout JLC, bukan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; Status FROZEN geometry; procurement PROVISIONAL -> FROZEN layout baseline; not production release; Supplier (none) -> JLCPCB; Supplier_URL https://shopee.co.id/product/119918417/25227825636 -> https://jlcpcb.com/partdetail/YAGEO-RC0805FR07330KL/C114528
- R22: Assembly (none) -> JLCPCB Standard planned; process review pending; Footprint_Status (none) -> Layout baseline reviewed; final PCB DRC/DFM and assembly re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; LCSC Part # (none) -> C96346; Manufacturer (none) -> Yageo; Procurement_Status PROVISIONAL - listing/candidate only; exact MPN and domesti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 -> FROZEN MPN/catalog identity; stock not reserved; order revi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; Selection_Note Sama dengan basis komponen HAV; tidak mengubah HAV. -> MPN dan footprint dipertahankan; baseline layout JLC, bukan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; Status FROZEN geometry; procurement PROVISIONAL -> FROZEN layout baseline; not production release; Supplier (none) -> JLCPCB; Supplier_URL https://shopee.co.id/product/16973105/49051878593 -> https://jlcpcb.com/partdetail/YAGEO-RC0805FR07100KL/C96346
