File: main_unit/main_rtc_i2c_oled.kicad_sch (KiCad schematic)
At the start: 11 parts, among them J3 OLED_SH1106_I2C, U3 DS3231SN#

Commit message: Sync HAV and WBV KiCad sources with JLCPCB review packages
Parts:
- BT1: value CR2032 + HOLDER -> CR2032 HOLDER; footprint (none) -> wbv_jlc:BatteryHolder_Keystone_1060TR_1x2032; Assembly (none) -> JLCPCB SMT assembly planned; holder/socket only; Footprint_Status (none) -> Manufacturer drawing reviewed; final placement DRC/DFM/CPL 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; LCSC Part # (none) -> C238069; MPN OPEN -> 1060TR; Manufacturer (none) -> Keystone Electronics; Package (none) -> SMT CR2032 holder 28.4x16mm H5.5mm; overall lead span31.9mm; Procurement_Status (none) -> FROZEN exact MPN/C-code; stock snapshot2026-10-06 not reser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; Selection_Note (none) -> 1060TR tape/reel holder only; same mechanical pattern as106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; Status PROVISIONAL - not for fabrication -> FROZEN layout baseline; not production release; Supplier (none) -> JLCPCB; Supplier_URL (none) -> https://jlcpcb.com/partdetail/Keystone-1060TR/C238069
- C13, C14: Assembly (none) -> JLCPCB Standard planned; process review pending; Footprint_Status (none) -> Layout baseline reviewed; final PCB DRC/DFM and assembly re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; LCSC Part # (none) -> C3018562; Manufacturer (none) -> KEMET; Procurement_Status PROVISIONAL - listing/candidate only; exact MPN and domesti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 -> FROZEN MPN/catalog identity; stock not reserved; order revi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; Selection_Note Sama dengan basis komponen HAV; tidak mengubah HAV. -> MPN dan footprint dipertahankan; baseline layout JLC, bukan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; Status FROZEN geometry; procurement PROVISIONAL -> FROZEN layout baseline; not production release; Supplier (none) -> JLCPCB; Supplier_URL https://shopee.co.id/product/25936178/8912815073 -> https://jlcpcb.com/partdetail/KEMET-C0805C104K5RACTU/C30185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
- C15: Assembly (none) -> JLCPCB Standard planned; process review pending; Footprint_Status (none) -> Layout baseline reviewed; final PCB DRC/DFM and assembly re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; LCSC Part # (none) -> C15850; Manufacturer (none) -> Samsung Electro-Mechanics; Procurement_Status PROVISIONAL - listing/candidate only; exact MPN and domesti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 -> FROZEN MPN/catalog identity; stock not reserved; order revi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; Selection_Note Samsung resmi: 2.0x1.25x1.25mm; cek effective C. Listing te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 -> MPN dan footprint dipertahankan; baseline layout JLC, bukan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; Status FROZEN geometry; procurement PROVISIONAL -> FROZEN layout baseline; not production release; Supplier (none) -> JLCPCB; Supplier_URL https://shopee.co.id/product/45119540/7441919037 -> https://jlcpcb.com/partdetail/CL21A106KAYNNNE/C15850
- J3: Assembly (none) -> JLCPCB Standard planned; process review pending; Footprint_Status (none) -> Layout baseline reviewed; final PCB DRC/DFM and assembly re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; LCSC Part # (none) -> C144395; Manufacturer (none) -> JST; Procurement_Status PROVISIONAL - listing/candidate only; exact MPN and domesti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 -> FROZEN MPN/catalog identity; stock not reserved; order revi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; Selection_Note Konektor kabel sisi PCB, bukan footprint board OLED/GPS. Wa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 -> MPN dan footprint dipertahankan; baseline layout JLC, bukan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; Status FROZEN geometry; procurement PROVISIONAL -> FROZEN layout baseline; not production release; Supplier (none) -> JLCPCB; Supplier_URL https://shopee.co.id/Connector-XH-2.54-PCB-Male-2P-3P-4P-5P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 -> https://jlcpcb.com/partdetail/JST-B4B_XH_A_LF_SN/C144395
- R17, R18: Assembly (none) -> JLCPCB Standard planned; process review pending; Footprint_Status (none) -> Layout baseline reviewed; final PCB DRC/DFM and assembly re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; LCSC Part # (none) -> C60816; Manufacturer (none) -> Yageo; Procurement_Status PROVISIONAL - listing/candidate only; exact MPN and domesti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 -> FROZEN MPN/catalog identity; stock not reserved; order revi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; Selection_Note Pilih varian nilai tepat; resistor generik bukan otomatis e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 -> MPN dan footprint dipertahankan; baseline layout JLC, bukan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; Status FROZEN geometry; procurement PROVISIONAL -> FROZEN layout baseline; not production release; Supplier (none) -> JLCPCB; Supplier_URL https://shopee.co.id/product/16973105/49051878593 -> https://jlcpcb.com/partdetail/YAGEO-RC0805FR074K7L/C60816
- U3: Assembly (none) -> JLCPCB Standard planned; process review pending; Footprint_Status (none) -> Layout baseline reviewed; final PCB DRC/DFM and assembly re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; LCSC Part # (none) -> C5369307; Manufacturer (none) -> Analog Devices; Procurement_Status PROVISIONAL - listing/candidate only; exact MPN and domesti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 -> FROZEN MPN/catalog identity; stock not reserved; order revi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; Selection_Note IC bare, bukan breakout RTC; pilihan holder BT1 terpisah ma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 -> DS3231SN# bare SOIC16W; BT1 Keystone1060TR holder/C238069. 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; Status FROZEN geometry; procurement PROVISIONAL -> FROZEN layout baseline; not production release; Supplier (none) -> JLCPCB; Supplier_URL https://shopee.co.id/product/92457567/5856889595 -> https://jlcpcb.com/partdetail/AnalogDevices-DS3231SN/C53693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
Other:
- note added: "OLED SH1106 | J3 XH4 | BT1 1060TR"
- note removed: "OLED SH1106 | J3 XH4 | BT1 holder HOLD"
